File: hardware/esp8266_room_monitor.sch (EAGLE design)
At the start: 28 parts, among them CN1 Power, IC1 REG1117, SW2 Config, U1 ESP-12, U2 OPAMP-DUAL

Commit message: Webconfig redesign (part)
Webconfig HTML page completely redesigned:
* Parameters are now organised as sections and subsections
* Sections are shown as UI tabs to simplify navigation
* Radio Buttons are replaced with Dropdown Lists to save space on page
* Unobvious parameters can have pop-up Tooltips

Internal changes:
* Webconfig HTML page is much faster to transmit
* Web-server does not occasionally reset connection anymore
* Webconfig HTML generation code is rewritten, making it easier to add
more parameters / sections / subsections to Webconfig HTML page
* EEPROM parameters saved in memory are reorganised making it easier to
add more parameters
Parts:
- JP4: value AM2302 -> AM2301
Changed lines of the file:
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@@
 <part name="R10" library="resistor" deviceset="R-EU_" device="M0805" value="10K"/>
 <part name="+3V7" library="supply1" deviceset="+3V3" device=""/>
-<part name="JP4" library="adafruit" deviceset="PINHD-1X3" device="" value="AM2302"/>
+<part name="JP4" library="adafruit" deviceset="PINHD-1X3" device="" value="AM2301"/>
 <part name="JP5" library="adafruit" deviceset="PINHD-1X3" device="" value="DS18B20"/>
 <part name="R12" library="resistor" deviceset="R-EU_" device="M0805" value="4K7"/>
